File: pcb/3x4-macropad.kicad_sch (KiCad schematic)
At the start: 54 parts, among them SW1 SW_Push, SW10 SW_Push, SW11 SW_Push, SW12 SW_Push, SW2 SW_Push, SW3 SW_Push, SW4 SW_Push, SW5 SW_Push, SW6 SW_Push, SW7 SW_Push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

Commit message: Fixed Bugs
Other:
- note added: "SSD1306 OLED display"
- note removed: "Header for SSD1306 OLED display"
Changed lines of the file:
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@@
     (effects (font (size 1.27 1.27)) (justify left bottom))
   )
-  (text "Underglow LEDs (WS2812b)" (at 248.735 176.9743 0)
+  (text "Underglow LEDs (WS2812b)" (at 238.76 165.1 0)
     (effects (font (size 1.27 1.27)) (justify left bottom))
   )
@@
     (effects (font (size 1.27 1.27)) (justify left bottom))
   )
-  (text "Header for SSD1306 OLED display" (at 21.59 111.76 0)
+  (text "SSD1306 OLED display" (at 25.4 111.76 0)
     (effects (font (size 1.27 1.27)) (justify left bottom))
   )
